File: PCBs/EC Breakout/SmartRock_EC.sch (EAGLE design)
At the start: 53 parts, among them IC2 TL074P, U1 ADS1115IDGST, U2 TPS60400DBVR

Commit message: Breakout Board Fix
Parts:
- removed CN4: (no value), adafruit:JST_2PIN-THM
- removed JP4: (no value), pinhead:PINHD-1X9
- removed R12, R13: 10k, rcl:R-US_R1206
- removed R16: (no value), adafruit:R-US_M1206
- removed SJ1, SJ2: (no value), jumper:SJ
- R17, R18, R19: value 10k -> 3.3k
Connections:
- removed net 3VO: JP4.2
- removed net FLT: JP4.8
- removed net INT: CN4.1, JP1.8, R16.1
- removed net N$6: JP5.2, SJ2.2
- removed net RDY: JP4.9
- net AIN3: no longer SJ1.1
- net GND: now also U$7.3; no longer CN4.2, JP4.3, U$7.2
- net GPIO10: no longer JP4.5, R17.1
- net GPIO11: no longer JP4.4
- net GPIO5: no longer R19.1
- net GPIO6: no longer JP4.7, R18.1
- net GPIO9: no longer JP4.6, REED.1
- net GPIOA0: now also R17.1
- net GPIOA1: now also R18.1
- net GPIOA2: now also R19.1
- net GPIOA5: now also REED.1; no longer SJ1.2, SJ2.1
- net SCL: now also U$7.2; no longer R12.2, U$7.3
- net SDA: now also U$7.1; no longer R13.2, U$7.4
- net VCC: now also U$7.4; no longer JP4.1, R12.1, R13.1, R16.2, U$7.1
Other:
- note removed: "CN4"
- note removed: "Thermocouple Header"
