File: PCB/4-pin_EC_Breakout/SmartRock_4-pin_EC_Breakout-v5.sch (EAGLE design)
At the start: 41 parts, among them CN2 JST_3PIN_2MM, CN5 JST_4PIN_2MM, U1 CD4060BPWR, U2 TL074CPWR, U3 TL074CPWR, U4 TL074CPWR, U5 ADS1115, U6+ MAX660MX/NOPB, X1 B4B-PH-K-S

Commit message: Board Rev. 5 Progress
getting closer to a finished board
Parts:
- removed CN1: (no value), adafruit:JST_2PIN-THM
- removed CN5: JST_4PIN_2MM, JSTconnector:JST_4PIN_2MM
- removed JP3: (no value), pinhead:PINHD-1X4
- removed X1: B4B-PH-K-S, 2_pin_JST:B4B-PH-K-S
- added JP2: (no value), pinhead:PINHD-1X4
- JP1: device pinhead:PINHD-1X2 -> pinhead:PINHD-1X4
Connections:
- net B: now also JP2.4; no longer JP3.4, X1.4
- net GND: now also JP1.3; no longer CN1.1, CN5.3, JP1.2
- net M: now also JP2.2; no longer JP3.2, X1.2
- net N: now also JP2.3; no longer JP3.3, X1.3
- net SCALE_A: now also JP2.1; no longer JP3.1, X1.1
- net SCL: now also JP1.2; no longer CN5.2
- net SDA: now also JP1.1; no longer CN5.1
- net VCC: now also JP1.4; no longer CN1.2, CN5.4, JP1.1
Other:
- note removed: "CN4"
- moved on the sheet: C1, C2, C3, C4, C5, D1, D2, D3, D4, JP4, JP5, JP6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
