File: PCB/4-pin_EC_Breakout/SmartRock_4-pin_EC_Breakout-v5.brd (EAGLE design)
At the start: 80 x 33 mm, 38 parts, among them CN2 JST_3PIN_2MM, U1 CD4060BPWR, U2 TL074CPWR, U3 TL074CPWR, U4 TL074CPWR, U5 ADS1115, U6+ MAX660MX/NOPB

Commit message: Fit 4-pin on two layers
New circuit is on two layers now, layout done. I need to go over it again and get the trace lengths to match where needed and I need to check for physical interference. So close I can smell it.
Parts:
- moved C3 26.2 mm to (30.2, 20.8)
- moved U6+ 25.4 mm to (35.3, 20.6)
- moved C5 17.7 mm to (33.5, 16.5), turned to 0 degrees
- moved R14 15.1 mm to (24.6, 26.2), turned to 90 degrees
- moved R13 11.4 mm to (22.1, 26.2), turned to 90 degrees
- moved R5 10.2 mm to (6.60, 18.5), turned to 180 degrees
- moved U3 7.92 mm to (13.3, 20.2)
- moved C4 7.50 mm to (19.1, 26.2), turned to 90 degrees
- moved R2 6.48 mm to (11.9, 30.2), turned to 0 degrees
- moved TUNING_RESISTOR 6.27 mm to (11.2, 14.2)
- moved R8 5.45 mm to (55.6, 18.3), turned to 270 degrees
- moved R15 5.09 mm to (55.9, 12.4), turned to 90 degrees
- moved R1 4.72 mm to (17.0, 30.2), turned to 180 degrees
- moved D1 4.19 mm to (45.2, 13.7)
- moved D2 4.19 mm to (45.2, 10.9)
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Routing:
- net VCC: track 0.00 -> 38.9 mm, vias 0 -> 4
- net SCL: track 46.3 -> 75.1 mm, vias 0 -> 2
- net -VCC: track 69.2 -> 41.9 mm, vias 2 -> 3
- net SDA: track 52.7 -> 78.9 mm, vias 0 -> 2
- net OUT4: track 0.65 -> 14.0 mm, vias 0 -> 2
- net CAP1: track 25.8 -> 13.0 mm
- net N$17: track 5.59 -> 15.6 mm
- net A: track 4.72 -> 14.5 mm, vias 0 -> 2
- net N$2: track 10.9 -> 19.8 mm, vias 0 -> 2
- net OUT2: track 11.1 -> 3.06 mm, vias 2 -> 0
- net OUT3B: track 8.43 -> 16.0 mm
- net N$4: track 14.2 -> 20.8 mm
- net OUT2B: track 13.5 -> 20.0 mm
- net OUT4B: track 2.54 -> 9.03 mm
- net N$6: track 11.0 -> 16.7 mm
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- added copper zone on layer 1, net GND
- added copper zone on layer 16, net VCC
- removed copper zone on layer 16, net GND
- removed copper zone on layer 1, net VCC

Commit message: Fix cap positons
Parts:
- moved C1 20.3 mm to (71.1, 3.05), turned to 0 degrees
- moved C2 20.0 mm to (65.8, 3.05), turned to 0 degrees
- moved D1 1.27 mm to (46.5, 13.7)
- moved D2 1.27 mm to (46.5, 10.9)
- moved D3 1.27 mm to (46.5, 19.6)
- moved D4 1.27 mm to (46.5, 16.8)
Routing:
- net CAP1: track 13.0 -> 26.7 mm, vias 0 -> 2
- net CAP2: track 15.7 -> 25.9 mm, vias 2 -> 4
- net N$4: track 20.8 -> 22.1 mm
- net OUT2B: track 20.0 -> 21.3 mm
- net N$6: track 16.7 -> 17.7 mm
- net OUT3B: track 16.0 -> 16.7 mm
Changed lines of the file:
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@@
 </autorouter>
 <elements>
-<element name="C1" library="adafruit" library_urn="urn:adsk.eagle:library:420" package="C025-024X044" package3d_urn="urn:adsk.eagle:package:6240324/1" value="1uF" x="53.086" y="12.446" smashed="yes" rot="R270"/>
-<element name="C2" library="adafruit" library_urn="urn:adsk.eagle:library:420" package="C025-024X044" package3d_urn="urn:adsk.eagle:package:6240324/1" value="1uF" x="52.832" y="18.288" smashed="yes" rot="R90"/>
+<element name="C1" library="adafruit" library_urn="urn:adsk.eagle:library:420" package="C025-024X044" package3d_urn="urn:adsk.eagle:package:6240324/1" value="1uF" x="71.12" y="3.048" smashed="yes"/>
+<element name="C2" library="adafruit" library_urn="urn:adsk.eagle:library:420" package="C025-024X044" package3d_urn="urn:adsk.eagle:package:6240324/1" value="1uF" x="65.786" y="3.048" smashed="yes"/>
 <element name="C3" library="adafruit" library_urn="urn:adsk.eagle:library:420" package="C025-024X044" package3d_urn="urn:adsk.eagle:package:6240324/1" value="1uF" x="30.226" y="20.828" smashed="yes" rot="R270"/>
 <element name="C4" library="adafruit" library_urn="urn:adsk.eagle:library:420" package="C1206" package3d_urn="urn:adsk.eagle:package:6240335/1" value="1nF" x="19.05" y="26.162" smashed="yes" rot="R90"/>
 <element name="C5" library="adafruit" library_urn="urn:adsk.eagle:library:420" package="C025-024X044" package3d_urn="urn:adsk.eagle:package:6240324/1" value="1uF" x="33.528" y="16.51" smashed="yes"/>
 <element name="CN2" library="JSTconnector" package="JST_3PIN_2MM" value="JST_3PIN_2MM" x="76.962" y="20.066" smashed="yes" rot="R90"/>
-<element name="D1" library="adafruit" library_urn="urn:adsk.eagle:library:420" package="DO41-10" package3d_urn="urn:adsk.eagle:package:6240344/1" value="1N4004" x="45.212" y="13.716" smashed="yes" rot="R180"/>
-<element name="D2" library="adafruit" library_urn="urn:adsk.eagle:library:420" package="DO41-10" package3d_urn="urn:adsk.eagle:package:6240344/1" value="1N4004" x="45.212" y="10.922" smashed="yes" rot="R180"/>
-<element name="D3" library="adafruit" library_urn="urn:adsk.eagle:library:420" package="DO41-10" package3d_urn="urn:adsk.eagle:package:6240344/1" value="1N4004" x="45.212" y="19.558" smashed="yes" rot="R180"/>
-<element name="D4" library="adafruit" library_urn="urn:adsk.eagle:library:420" package="DO41-10" package3d_urn="urn:adsk.eagle:package:6240344/1" value="1N4004" x="45.212" y="16.764" smashed="yes" rot="R180"/>
+<element name="D1" library="adafruit" library_urn="urn:adsk.eagle:library:420" package="DO41-10" package3d_urn="urn:adsk.eagle:package:6240344/1" value="1N4004" x="46.482" y="13.716" smashed="yes" rot="R180"/>
+<element name="D2" library="adafruit" library_urn="urn:adsk.eagle:library:420" package="DO41-10" package3d_urn="urn:adsk.eagle:package:6240344/1" value="1N4004" x="46.482" y="10.922" smashed="yes" rot="R180"/>
+<element name="D3" library="adafruit" library_urn="urn:adsk.eagle:library:420" package="DO41-10" package3d_urn="urn:adsk.eagle:package:6240344/1" value="1N4004" x="46.482" y="19.558" smashed="yes" rot="R180"/>
+<element name="D4" library="adafruit" library_urn="urn:adsk.eagle:library:420" package="DO41-10" package3d_urn="urn:adsk.eagle:package:6240344/1" value="1N4004" x="46.482" y="16.764" smashed="yes" rot="R180"/>
 <element name="JP2" library="pinhead" library_urn="urn:adsk.eagle:library:325" package="1X04" package3d_urn="urn:adsk.eagle:package:22407/2" value="" x="2.032" y="22.098" smashed="yes" rot="R270">
 <attribute name="POPULARITY" value="91" x="-48.768" y="-7.112" size="1.778" layer="27" rot="R270" display="off"/>
@@
 <via x="67.3895" y="14.22845" extent="1-16" drill="0.35"/>
 <wire x1="67.3895" y1="14.22845" x2="67.3895" y2="11.5095" width="0.3048" layer="16"/>
-<wire x1="67.31" y1="11.43" x2="67.3895" y2="11.5095" width="0.3048" layer="16"/>
 <via x="67.3895" y="11.5095" extent="1-16" drill="0.35"/>
 <wire x1="67.3895" y1="11.5095" x2="59.69" y2="3.81" width="0.3048" layer="1"/>
@@
 <contactref element="D1" pad="A"/>
 <contactref element="U4" pad="6"/>
+<wire x1="41.402" y1="13.716" x2="40.132" y2="13.716" width="0.3048" layer="1"/>
 <wire x1="40.132" y1="13.716" x2="35.052" y2="8.636" width="0.3048" layer="1"/>
 <wire x1="22.022" y1="10.13" x2="23.144" y2="10.13" width="0.3048" layer="1"/>
@@
 <contactref element="R15" pad="2"/>
 <contactref element="U5" pad="AIN0"/>
-<wire x1="50.292" y1="10.922" x2="50.292" y2="13.716" width="0.3048" layer="1"/>
-<wire x1="50.292" y1="13.716" x2="53.086" y2="13.716" width="0.3048" layer="1"/>
-<wire x1="53.086" y1="13.716" x2="53.216" y2="13.846" width="0.3048" layer="1"/>
-<wire x1="53.216" y1="13.846" x2="55.88" y2="13.846" width="0.3048" layer="1"/>
+<wire x1="51.562" y1="10.922" x2="51.562" y2="13.716" width="0.3048" layer="1"/>
 <wire x1="55.88" y1="13.846" x2="58.544" y2="13.846" width="0.3048" layer="1"/>
 <wire x1="59.198" y1="13.192" x2="60.21" y2="13.192" width="0.3048" layer="1"/>
 <wire x1="58.544" y1="13.846" x2="59.198" y2="13.192" width="0.3048" layer="1"/>
+<wire x1="51.562" y1="13.716" x2="51.692" y2="13.846" width="0.3048" layer="1"/>
+<wire x1="51.692" y1="13.846" x2="55.88" y2="13.846" width="0.3048" layer="1"/>
+<via x="65.278" y="7.62" extent="1-16" drill="0.35"/>
+<wire x1="65.278" y1="7.62" x2="62.484" y2="10.414" width="0.3048" layer="16"/>
+<wire x1="62.484" y1="10.414" x2="62.484" y2="12.192" width="0.3048" layer="16"/>
+<via x="62.484" y="12.192" extent="1-16" drill="0.35"/>
+<wire x1="62.484" y1="12.192" x2="61.484" y2="13.192" width="0.3048" layer="1"/>
+<wire x1="61.484" y1="13.192" x2="60.21" y2="13.192" width="0.3048" layer="1"/>
+<wire x1="69.85" y1="3.048" x2="65.278" y2="7.62" width="0.3048" layer="1"/>
 </signal>
 <signal name="OUT2B">
 <contactref element="D2" pad="A"/>
 <contactref element="U4" pad="7"/>
-<wire x1="40.132" y1="10.922" x2="38.608" y2="10.922" width="0.3048" layer="1"/>
-<wire x1="38.608" y1="10.922" x2="35.56" y2="7.874" width="0.3048" layer="1"/>
+<wire x1="41.402" y1="10.922" x2="39.878" y2="10.922" width="0.3048" layer="1"/>
+<wire x1="39.878" y1="10.922" x2="36.83" y2="7.874" width="0.3048" layer="1"/>
 <wire x1="23.628" y1="7.874" x2="22.022" y2="9.48" width="0.3048" layer="1"/>
-<wire x1="35.56" y1="7.874" x2="23.628" y2="7.874" width="0.3048" layer="1"/>
+<wire x1="36.83" y1="7.874" x2="23.628" y2="7.874" width="0.3048" layer="1"/>
 </signal>
 <signal name="N$5">
@@
 <contactref element="U4" pad="9"/>
 <contactref element="D3" pad="A"/>
-<wire x1="40.132" y1="19.558" x2="40.132" y2="18.796" width="0.3048" layer="1"/>
-<wire x1="40.132" y1="18.796" x2="31.466" y2="10.13" width="0.3048" layer="1"/>
-<wire x1="31.466" y1="10.13" x2="27.762" y2="10.13" width="0.3048" layer="1"/>
+<wire x1="41.402" y1="19.558" x2="41.402" y2="19.304" width="0.3048" layer="1"/>
+<wire x1="41.402" y1="19.304" x2="32.228" y2="10.13" width="0.3048" layer="1"/>
+<wire x1="32.228" y1="10.13" x2="27.762" y2="10.13" width="0.3048" layer="1"/>
 </signal>
 <signal name="CAP2">
@@
 <contactref element="R8" pad="2"/>
 <contactref element="U5" pad="AIN1"/>
-<wire x1="50.292" y1="19.558" x2="50.292" y2="16.764" width="0.3048" layer="1"/>
-<wire x1="50.292" y1="16.764" x2="50.546" y2="17.018" width="0.3048" layer="1"/>
-<wire x1="50.546" y1="17.018" x2="52.832" y2="17.018" width="0.3048" layer="1"/>
-<wire x1="52.832" y1="17.018" x2="55.496" y2="17.018" width="0.3048" layer="1"/>
-<wire x1="55.496" y1="17.018" x2="55.626" y2="16.888" width="0.3048" layer="1"/>
+<wire x1="51.562" y1="19.558" x2="51.562" y2="16.764" width="0.3048" layer="1"/>
 <wire x1="55.626" y1="16.888" x2="55.756" y2="16.888" width="0.3048" layer="1"/>
-<wire x1="55.756" y1="16.888" x2="57.912" y2="14.732" width="0.3048" layer="1"/>
+<wire x1="55.756" y1="16.888" x2="55.88" y2="16.764" width="0.3048" layer="1"/>
 <via x="57.912" y="14.732" extent="1-16" drill="0.35"/>
+<wire x1="55.88" y1="16.764" x2="57.912" y2="14.732" width="0.3048" layer="1"/>
 <wire x1="57.912" y1="14.732" x2="57.912" y2="12.954" width="0.3048" layer="16"/>
 <via x="57.912" y="12.954" extent="1-16" drill="0.35"/>
@@
 <wire x1="58.02741875" y1="12.954" x2="58.25296875" y2="12.72845" width="0.3048" layer="1"/>
 <wire x1="58.25296875" y1="12.72845" x2="60.17355" y2="12.72845" width="0.3048" layer="1"/>
+<wire x1="51.562" y1="16.764" x2="55.88" y2="16.764" width="0.3048" layer="1"/>
+<wire x1="60.198" y1="12.68" x2="60.21" y2="12.692" width="0.3048" layer="1"/>
+<wire x1="64.516" y1="3.048" x2="64.516" y2="5.588" width="0.3048" layer="1"/>
+<wire x1="64.516" y1="5.588" x2="63.754" y2="6.35" width="0.3048" layer="1"/>
+<via x="63.754" y="6.35" extent="1-16" drill="0.35"/>
+<wire x1="63.754" y1="6.35" x2="60.198" y2="9.906" width="0.3048" layer="16"/>
+<wire x1="60.198" y1="9.906" x2="60.198" y2="11.43" width="0.3048" layer="16"/>
+<via x="60.198" y="11.43" extent="1-16" drill="0.35"/>
+<wire x1="60.198" y1="11.43" x2="60.198" y2="12.68" width="0.3048" layer="1"/>
 </signal>
 <signal name="OUT3B">
 <contactref element="U4" pad="8"/>
 <contactref element="D4" pad="A"/>
-<wire x1="40.132" y1="16.764" x2="40.132" y2="15.748" width="0.3048" layer="1"/>
-<wire x1="40.132" y1="15.748" x2="33.864" y2="9.48" width="0.3048" layer="1"/>
+<wire x1="41.402" y1="16.764" x2="41.148" y2="16.764" width="0.3048" layer="1"/>
+<wire x1="41.148" y1="16.764" x2="33.864" y2="9.48" width="0.3048" layer="1"/>
 <wire x1="33.864" y1="9.48" x2="27.762" y2="9.48" width="0.3048" layer="1"/>
 </signal>
